Commit message: add real slam

File: src/tracer_jaka/tracer_jaka_mujoco/urdf/tracer_jaka_zu5.urdf (robot description, URDF)
Before this commit: robot tracer_jaka_zu5, 33 links, 32 joints
Links:
- removed link laser_frame
- added link laser_link; visual mesh filename=package://tracer_jaka_mujoco/urdf/meshes/laser.STL scale=0.001 0.001 0.001
- link imu_link: geometry visual mesh filename=package://tracer_jaka_mujoco/urdf/meshes/imu.STL scale=0.001 0.001 0.001
Joints:
- joint base_to_imu: origin xyz=0.20 0.15 0.255 rpy=0 0 0 -> xyz=0.185 0.185 0.23 rpy=0 0 3.1415
- joint base_to_laser: child laser_frame -> laser_link; origin xyz=0.29 0 0.26 rpy=0 0 0 -> xyz=0.31 0 0.03 rpy=0 0 0

File: src/tracer_jaka/tracer_jaka_mujoco/urdf/tracer_jaka_zu5_real.urdf (robot description, URDF)
Before this commit: robot tracer_jaka_zu5, 33 links, 32 joints
Links:
- removed link laser_frame
- added link laser_link; visual mesh filename=package://tracer_jaka_mujoco/urdf/meshes/laser.STL scale=0.001 0.001 0.001
- link imu_link: geometry visual mesh filename=package://tracer_jaka_mujoco/urdf/meshes/imu.STL scale=0.001 0.001 0.001
Joints:
- joint base_footprint_to_base_link: origin xyz=0 0 0.136 rpy=0 0 0 -> xyz=0 0 0.147 rpy=0 0 0
- joint base_to_imu: origin xyz=0.20 0.15 0.255 rpy=0 0 0 -> xyz=0.185 0.185 0.23 rpy=0 0 3.1415
- joint base_to_laser: child laser_frame -> laser_link; origin xyz=0.29 0 0.26 rpy=0 0 0 -> xyz=0.31 0 0.03 rpy=0 0 0

Commit message: add d455

File: src/tracer_jaka/tracer_jaka_mujoco/urdf/tracer_jaka_zu5.urdf (robot description, URDF)
Before this commit: robot tracer_jaka_zu5, 33 links, 32 joints
Links:
- added link d455_link; visual mesh filename=package://tracer_jaka_mujoco/urdf/meshes/d455.STL scale=0.001 0.001 0.001
Joints:
- added joint base_to_d455: type fixed, parent base_link, child d455_link, origin xyz=0.25 0 0.24 rpy=1.5708 0 1.5708

Commit message: fixed some bug

File: src/tracer_jaka/tracer_jaka_mujoco/urdf/tracer_jaka_zu5.urdf (robot description, URDF)
Before this commit: robot tracer_jaka_zu5, 34 links, 33 joints
Joints:
- joint base_to_d455: origin xyz=0.25 0 0.24 rpy=1.5708 0 1.5708 -> xyz=0.25 0 0.24 rpy=0 0 0
