Commit message: feat: add C++ localization readiness and self-collision checks
Add selectable Cartographer mapping and localization with planner readiness gating. Rename localization and trajectory bridge packages, update tool0 orientation, and document usage.

File: src/robotics/tracer_jaka_description/urdf/tracer_jaka_zu5.urdf (robot description, URDF)
Before this commit: robot tracer_jaka_zu5, 34 links, 33 joints
Joints:
- joint tool0_joint: origin xyz=0 0 0.27 rpy=0 0 0 -> xyz=0 0 0.27 rpy=0 0 3.141592653589793
